File: rbpi_can.kicad_pcb (KiCad board)
At the start: 2 copper layers, 12 parts, among them P1 CONN, P2 RBPI_HEADER, U1 OKI-78SR, U2 MCP2551, U3 MCP2515, Y1 10MHZ

Commit message: Clean up project
Other:
- board outline added: 31.8 x 54.6 mm
Changed lines of the file:
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@@
     (links 41)
     (no_connects 0)
-    (area 129.54 89.9816 161.290001 144.8184)
+    (area 129.464999 90.094999 161.365001 144.855001)
     (thickness 1.6)
-    (drawings 0)
+    (drawings 4)
     (tracks 72)
     (zones 0)
@@
   )
   (setup
-    (last_trace_width 0.635)
+    (last_trace_width 0.1524)
     (user_trace_width 0.254)
     (user_trace_width 0.381)
@@
     (uvia_min_drill 0)
     (pcb_text_width 0.3)
-    (pcb_text_size 1.5 1.5)
+    (pcb_text_size 1 1)
     (mod_edge_width 0.15)
-    (mod_text_size 1 1)
-    (mod_text_width 0.15)
+    (mod_text_size 0.6 0.6)
+    (mod_text_width 0.1)
     (pad_size 1.524 1.524)
     (pad_drill 0.762)
@@
     (visible_elements FFFFFF7F)
     (pcbplotparams
-      (layerselection 0x00030_80000001)
-      (usegerberextensions false)
+      (layerselection 0x010f0_80000001)
+      (usegerberextensions true)
       (excludeedgelayer true)
       (linewidth 0.100000)
@@
     (tags "capacitor 1206")
     (attr smd)
-    (fp_text reference C1 (at -4.445 0 360) (layer F.SilkS)
-      (effects (font (size 1 1) (thickness 0.15)))
-    )
-    (fp_text value 22p (at 0.127 -2.159 270) (layer F.Fab)
-      (effects (font (size 1 1) (thickness 0.15)))
+    (fp_text reference C1 (at -4.064 0 360) (layer F.SilkS)
+      (effects (font (size 0.6 0.6) (thickness 0.1)))
+    )
+    (fp_text value 22p (at -4.064 -2.032 360) (layer F.Fab)
+      (effects (font (size 0.6 0.6) (thickness 0.1)))
     )
     (fp_line (start -3.3 -1.15) (end 3.3 -1.15) (layer F.CrtYd) (width 0.05))
@@
     (tags "capacitor 1206")
     (attr smd)
-    (fp_text reference C2 (at -4.064 -0.127 180) (layer F.SilkS)
-      (effects (font (size 1 1) (thickness 0.15)))
-    )
-    (fp_text value 22p (at 0 2.3 90) (layer F.Fab)
-      (effects (font (size 1 1) (thickness 0.15)))
+    (fp_text reference C2 (at -4.064 0 180) (layer F.SilkS)
+      (effects (font (size 0.6 0.6) (thickness 0.1)))
+    )
+    (fp_text value 22p (at -4.064 2.159 180) (layer F.Fab)
+      (effects (font (size 0.6 0.6) (thickness 0.1)))
     )
     (fp_line (start -3.3 -1.15) (end 3.3 -1.15) (layer F.CrtYd) (width 0.05))
@@
     (descr "Through hole pin header")
     (tags "pin header")
-    (fp_text reference P1 (at 0 15.494) (layer F.SilkS)
-      (effects (font (size 1 1) (thickness 0.15)))
-    )
-    (fp_text value CONN (at 0 -2.794) (layer F.Fab)
-      (effects (font (size 1 1) (thickness 0.15)))
+    (fp_text reference P1 (at 0 15.24) (layer F.SilkS)
+      (effects (font (size 0.6 0.6) (thickness 0.1)))
+    )
+    (fp_text value CONN (at 0 -2.54) (layer F.Fab)
+      (effects (font (size 0.6 0.6) (thickness 0.1)))
     )
     (fp_line (start -1.75 -1.75) (end -1.75 14.45) (layer F.CrtYd) (width 0.05))
@@
     (descr "Through hole pin header")
     (tags "pin header")
-    (fp_text reference P2 (at 1.016 -2.286) (layer F.SilkS)
-      (effects (font (size 1 1) (thickness 0.15)))
-    )
-    (fp_text value RBPI_HEADER (at -2.032 14.732 90) (layer F.Fab)
-      (effects (font (size 1 1) (thickness 0.15)))
+    (fp_text reference P2 (at 1.27 24.13 180) (layer F.SilkS)
+      (effects (font (size 0.6 0.6) (thickness 0.1)))
+    )
+    (fp_text value RBPI_HEADER (at -2.54 42.926 90) (layer F.Fab)
+      (effects (font (size 0.6 0.6) (thickness 0.1)))
     )
     (fp_line (start -1.75 -1.75) (end -1.75 50.05) (layer F.CrtYd) (width 0.05))
@@
     (attr smd)
     (fp_text reference R1 (at 4.191 0 360) (layer F.SilkS)
-      (effects (font (size 1 1) (thickness 0.15)))
-    )
-    (fp_text value 1k (at 0 2.3 270) (layer F.Fab)
-      (effects (font (size 1 1) (thickness 0.15)))
+      (effects (font (size 0.6 0.6) (thickness 0.1)))
+    )
+    (fp_text value 1k (at -4.064 0 540) (layer F.Fab)
+      (effects (font (size 0.6 0.6) (thickness 0.1)))
     )
     (fp_line (start -3.3 -1.2) (end 3.3 -1.2) (layer F.CrtYd) (width 0.05))
@@
     (attr smd)
     (fp_text reference R2 (at 4.191 0 360) (layer F.SilkS)
-      (effects (font (size 1 1) (thickness 0.15)))
-    )
-    (fp_text value 10k (at -4.953 0 270) (layer F.Fab)
-      (effects (font (size 1 1) (thickness 0.15)))
+      (effects (font (size 0.6 0.6) (thickness 0.1)))
+    )
+    (fp_text value 10k (at -4.064 0 360) (layer F.Fab)
+      (effects (font (size 0.6 0.6) (thickness 0.1)))
     )
     (fp_line (start -3.3 -1.2) (end 3.3 -1.2) (layer F.CrtYd) (width 0.05))
@@
     (attr smd)
     (fp_text reference R3 (at -4.191 0 180) (layer F.SilkS)
-      (effects (font (size 1 1) (thickness 0.15)))
-    )
-    (fp_text value 18k (at 4.826 0 90) (layer F.Fab)
-      (effects (font (size 1 1) (thickness 0.15)))
+      (effects (font (size 0.6 0.6) (thickness 0.1)))
+    )
+    (fp_text value 18k (at 4.064 0 180) (layer F.Fab)
+      (effects (font (size 0.6 0.6) (thickness 0.1)))
     )
     (fp_line (start -3.3 -1.2) (end 3.3 -1.2) (layer F.CrtYd) (width 0.05))
@@
     (attr smd)
     (fp_text reference R4 (at 4.191 0 360) (layer F.SilkS)
-      (effects (font (size 1 1) (thickness 0.15)))
-    )
-    (fp_text value 120 (at 0 2.3 270) (layer F.Fab)
-      (effects (font (size 1 1) (thickness 0.15)))
+      (effects (font (size 0.6 0.6) (thickness 0.1)))
+    )
+    (fp_text value 120 (at -3.937 -0.127 360) (layer F.Fab)
+      (effects (font (size 0.6 0.6) (thickness 0.1)))
     )
     (fp_line (start -3.3 -1.2) (end 3.3 -1.2) (layer F.CrtYd) (width 0.05))
@@
   (module footprints:OKI-78SR (layer F.Cu)
     (at 144.399 104.521 180)
-    (fp_text reference U1 (at -0.381 8.128 180) (layer F.SilkS)
-      (effects (font (size 1 1) (thickness 0.15)))
-    )
-    (fp_text value OKI-78SR (at 0.127 6.35 180) (layer F.Fab)
-      (effects (font (size 1 1) (thickness 0.15)))
+    (fp_text reference U1 (at 0.127 7.747 180) (layer F.SilkS)
+      (effects (font (size 0.6 0.6) (thickness 0.1)))
+    )
+    (fp_text value OKI-78SR (at -0.381 13.462 180) (layer F.Fab)
+      (effects (font (size 0.6 0.6) (thickness 0.1)))
     )
     (fp_line (start 8.255 2.413) (end 8.255 12.827) (layer F.SilkS) (width 0.15))
@@
     (descr "8-lead dip package, row spacing 7.62 mm (300 mils)")
     (tags "dil dip 2.54 300")
-    (fp_text reference U2 (at 3.81 6.477) (layer F.SilkS)
-      (effects (font (size 1 1) (thickness 0.15)))
-    )
-    (fp_text value MCP2551 (at 3.81 3.81) (layer F.Fab)
-      (effects (font (size 1 1) (thickness 0.15)))
+    (fp_text reference U2 (at 3.683 4.191) (layer F.SilkS)
+      (effects (font (size 0.6 0.6) (thickness 0.1)))
+    )
+    (fp_text value MCP2551 (at 3.429 -3.175) (layer F.Fab)
+      (effects (font (size 0.6 0.6) (thickness 0.1)))
     )
     (fp_line (start -1.05 -2.45) (end -1.05 10.1) (layer F.CrtYd) (width 0.05))
@@
     (descr "18-lead dip package, row spacing 7.62 mm (300 mils)")
     (tags "dil dip 2.54 300")
-    (fp_text reference U3 (at 3.81 5.334) (layer F.SilkS)
-      (effects (font (size 1 1) (thickness 0.15)))
-    )
-    (fp_text value MCP2515 (at 3.81 1.27) (layer F.Fab)
-      (effects (font (size 1 1) (thickness 0.15)))
+    (fp_text reference U3 (at 3.81 10.16) (layer F.SilkS)
+      (effects (font (size 0.6 0.6) (thickness 0.1)))
+    )
+    (fp_text value MCP2515 (at 3.683 23.495) (layer F.Fab)
+      (effects (font (size 0.6 0.6) (thickness 0.1)))
     )
     (fp_line (start -1.05 -2.45) (end -1.05 22.8) (layer F.CrtYd) (width 0.05))
@@
     (descr "Crystal, Quarz, HC49/U, vertical, stehend,")
     (tags "Crystal, Quarz, HC49/U, vertical, stehend,")
-    (fp_text reference Y1 (at -6.604 0 360) (layer F.SilkS)
-      (effects (font (size 1 1) (thickness 0.15)))
-    )
-    (fp_text value 10MHZ (at -8.382 0 360) (layer F.Fab)
-      (effects (font (size 1 1) (thickness 0.15)))
+    (fp_text reference Y1 (at 0.127 0 360) (layer F.SilkS)
+      (effects (font (size 0.6 0.6) (thickness 0.1)))
+    )
+    (fp_text value 10MHZ (at -6.35 0 360) (layer F.Fab)
+      (effects (font (size 0.6 0.6) (thickness 0.1)))
     )
     (fp_line (start 4.699 -1.00076) (end 4.89966 -0.59944) (layer F.SilkS) (width 0.15))
@@
       (net 2 "Net-(C2-Pad1)"))
   )
+  (gr_line (start 129.54 90.17) (end 161.29 90.17) (angle 90) (layer Edge.Cuts) (width 0.15))
+  (gr_line (start 129.54 144.78) (end 129.54 90.17) (angle 90) (layer Edge.Cuts) (width 0.15))
+  (gr_line (start 161.29 144.78) (end 129.54 144.78) (angle 90) (layer Edge.Cuts) (width 0.15))
+  (gr_line (start 161.29 90.17) (end 161.29 144.78) (angle 90) (layer Edge.Cuts) (width 0.15))
   (segment (start 131.826 130.461) (end 132.64794 130.461) (width 0.635) (layer F.Cu) (net 1))
   (segment (start 132.64794 130.461) (end 136.271 134.08406) (width 0.635) (layer F.Cu) (net 1))
