File: rpi_can.kicad_pcb (KiCad board)
At the start: 2 copper layers, 31.8 x 54.6 mm, 12 parts, among them P1 CONN, P2 RBPI_HEADER, U1 OKI-78SR, U2 MCP2551, U3 MCP2515, Y1 10MHZ

Commit message: Rename files
Other:
- board text added: "CANH"
- board text added: "CANL"
- board text added: "GND"
- board text added: "VI"
- board text added: "VO"
Changed lines of the file:
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@@
     (area 129.464999 90.094999 161.365001 144.855001)
     (thickness 1.6)
-    (drawings 4)
+    (drawings 10)
     (tracks 72)
     (zones 0)
@@
     (uvia_min_size 0)
     (uvia_min_drill 0)
-    (pcb_text_width 0.3)
-    (pcb_text_size 1 1)
+    (pcb_text_width 0.1)
+    (pcb_text_size 0.6 0.6)
     (mod_edge_width 0.15)
     (mod_text_size 0.6 0.6)
@@
     (tags "capacitor 1206")
     (attr smd)
-    (fp_text reference C1 (at -4.064 0 360) (layer F.SilkS)
-      (effects (font (size 0.6 0.6) (thickness 0.1)))
-    )
-    (fp_text value 22p (at -4.064 -2.032 360) (layer F.Fab)
+    (fp_text reference C1 (at -3.937 0.889 360) (layer F.SilkS)
+      (effects (font (size 0.6 0.6) (thickness 0.1)))
+    )
+    (fp_text value 22p (at -3.937 -1.016 360) (layer F.SilkS)
       (effects (font (size 0.6 0.6) (thickness 0.1)))
     )
@@
     (tags "capacitor 1206")
     (attr smd)
-    (fp_text reference C2 (at -4.064 0 180) (layer F.SilkS)
-      (effects (font (size 0.6 0.6) (thickness 0.1)))
-    )
-    (fp_text value 22p (at -4.064 2.159 180) (layer F.Fab)
+    (fp_text reference C2 (at -4.064 -0.889 180) (layer F.SilkS)
+      (effects (font (size 0.6 0.6) (thickness 0.1)))
+    )
+    (fp_text value 22p (at -4.064 1.016 180) (layer F.SilkS)
       (effects (font (size 0.6 0.6) (thickness 0.1)))
     )
@@
     (descr "Through hole pin header")
     (tags "pin header")
-    (fp_text reference P2 (at 1.27 24.13 180) (layer F.SilkS)
-      (effects (font (size 0.6 0.6) (thickness 0.1)))
-    )
-    (fp_text value RBPI_HEADER (at -2.54 42.926 90) (layer F.Fab)
+    (fp_text reference P2 (at 1.27 50.673 180) (layer F.SilkS)
+      (effects (font (size 0.6 0.6) (thickness 0.1)))
+    )
+    (fp_text value RBPI_HEADER (at -2.413 44.831 90) (layer F.Fab)
       (effects (font (size 0.6 0.6) (thickness 0.1)))
     )
@@
       (effects (font (size 0.6 0.6) (thickness 0.1)))
     )
-    (fp_text value 1k (at -4.064 0 540) (layer F.Fab)
+    (fp_text value 1k (at -4.064 0 360) (layer F.SilkS)
       (effects (font (size 0.6 0.6) (thickness 0.1)))
     )
@@
       (effects (font (size 0.6 0.6) (thickness 0.1)))
     )
-    (fp_text value 10k (at -4.064 0 360) (layer F.Fab)
+    (fp_text value 10k (at -4.064 0 360) (layer F.SilkS)
       (effects (font (size 0.6 0.6) (thickness 0.1)))
     )
@@
       (effects (font (size 0.6 0.6) (thickness 0.1)))
     )
-    (fp_text value 18k (at 4.064 0 180) (layer F.Fab)
+    (fp_text value 18k (at 4.064 0 180) (layer F.SilkS)
       (effects (font (size 0.6 0.6) (thickness 0.1)))
     )
@@
       (effects (font (size 0.6 0.6) (thickness 0.1)))
     )
-    (fp_text value 120 (at -3.937 -0.127 360) (layer F.Fab)
+    (fp_text value 120 (at -3.937 -0.127 360) (layer F.SilkS)
       (effects (font (size 0.6 0.6) (thickness 0.1)))
     )
@@
     )
   )
-  (module footprints:OKI-78SR (layer F.Cu)
-    (at 144.399 104.521 180)
-    (fp_text reference U1 (at 0.127 7.747 180) (layer F.SilkS)
-      (effects (font (size 0.6 0.6) (thickness 0.1)))
-    )
-    (fp_text value OKI-78SR (at -0.381 13.462 180) (layer F.Fab)
-      (effects (font (size 0.6 0.6) (thickness 0.1)))
-    )
-    (fp_line (start 8.255 2.413) (end 8.255 12.827) (layer F.SilkS) (width 0.15))
-    (fp_line (start 8.255 12.827) (end -8.255 12.827) (layer F.SilkS) (width 0.15))
-    (fp_line (start -8.255 12.827) (end -8.255 2.413) (layer F.SilkS) (width 0.15))
-    (fp_line (start -8.255 2.413) (end 8.255 2.413) (layer F.SilkS) (width 0.15))
-    (pad 3 thru_hole circle (at 6.985 10.16) (size 2.032 2.032) (drill 0.8128) (layers *.Cu *.Mask F.SilkS)
-      (net 6 VDD))
-    (pad 1 thru_hole circle (at 6.985 5.08) (size 2.032 2.032) (drill 0.8128) (layers *.Cu *.Mask F.SilkS)
-      (net 3 "Net-(P1-Pad1)"))
-    (pad 2 thru_hole oval (at 6.985 7.62) (size 2.032 2.032) (drill 0.8128) (layers *.Cu *.Mask F.SilkS)
-      (net 4 GND))
-  )
   (module Housings_DIP:DIP-8_W7.62mm (layer F.Cu)
     (at 140.589 107.061)
@@
       (effects (font (size 0.6 0.6) (thickness 0.1)))
     )
-    (fp_text value MCP2551 (at 3.429 -3.175) (layer F.Fab)
+    (fp_text value MCP2551 (at 3.429 -3.175) (layer F.SilkS)
       (effects (font (size 0.6 0.6) (thickness 0.1)))
     )
@@
       (effects (font (size 0.6 0.6) (thickness 0.1)))
     )
-    (fp_text value MCP2515 (at 3.683 23.495) (layer F.Fab)
+    (fp_text value MCP2515 (at 3.683 23.495) (layer F.SilkS)
       (effects (font (size 0.6 0.6) (thickness 0.1)))
     )
@@
       (effects (font (size 0.6 0.6) (thickness 0.1)))
     )
-    (fp_text value 10MHZ (at -6.35 0 360) (layer F.Fab)
+    (fp_text value 10MHZ (at -6.35 0 360) (layer F.SilkS)
       (effects (font (size 0.6 0.6) (thickness 0.1)))
     )
@@
       (net 2 "Net-(C2-Pad1)"))
   )
+  (module footprints:OKI-78SR (layer F.Cu)
+    (at 144.399 104.521 180)
+    (fp_text reference U1 (at -0.254 7.747 180) (layer F.SilkS)
+      (effects (font (size 0.6 0.6) (thickness 0.1)))
+    )
+    (fp_text value OKI-78SR (at 0.127 13.462 180) (layer F.SilkS)
+      (effects (font (size 0.6 0.6) (thickness 0.1)))
+    )
+    (fp_line (start 8.255 2.413) (end 8.255 12.827) (layer F.SilkS) (width 0.15))
+    (fp_line (start 8.255 12.827) (end -8.255 12.827) (layer F.SilkS) (width 0.15))
+    (fp_line (start -8.255 12.827) (end -8.255 2.413) (layer F.SilkS) (width 0.15))
+    (fp_line (start -8.255 2.413) (end 8.255 2.413) (layer F.SilkS) (width 0.15))
+    (pad 3 thru_hole oval (at 6.985 10.16) (size 2.032 1.524) (drill 0.8128) (layers *.Cu *.Mask F.SilkS)
+      (net 6 VDD))
+    (pad 1 thru_hole oval (at 6.985 5.08) (size 2.032 1.524) (drill 0.8128) (layers *.Cu *.Mask F.SilkS)
+      (net 3 "Net-(P1-Pad1)"))
+    (pad 2 thru_hole oval (at 6.985 7.62) (size 2.032 1.524) (drill 0.8128) (layers *.Cu *.Mask F.SilkS)
+      (net 4 GND))
+  )
+  (gr_text CANL (at 130.175 108.458 270) (layer F.SilkS)
+    (effects (font (size 0.6 0.6) (thickness 0.1)))
+  )
+  (gr_text "CANH\n" (at 130.175 105.791 270) (layer F.SilkS)
+    (effects (font (size 0.6 0.6) (thickness 0.1)))
+  )
+  (gr_text GND (at 130.175 103.251 270) (layer F.SilkS)
+    (effects (font (size 0.6 0.6) (thickness 0.1)))
+  )
+  (gr_text VO (at 130.175 100.711 270) (layer F.SilkS)
+    (effects (font (size 0.6 0.6) (thickness 0.1)))
+  )
+  (gr_text GND (at 130.175 98.044 270) (layer F.SilkS)
+    (effects (font (size 0.6 0.6) (thickness 0.1)))
+  )
+  (gr_text VI (at 130.175 95.758 270) (layer F.SilkS)
+    (effects (font (size 0.6 0.6) (thickness 0.1)))
+  )
   (gr_line (start 129.54 90.17) (end 161.29 90.17) (angle 90) (layer Edge.Cuts) (width 0.15))
